File: banana2header.kicad_pcb (KiCad board)
At the start: 2 copper layers, 35 x 50 mm, 6 parts, among them J1 Conn_01x01_Female, J2 Conn_01x01_Female, J3 Conn_01x01_Female, J4 Molex_SL_01x03_Male, J5 Conn_01x02_Male, J6 Conn_01x02_Male

Commit message: add license decal
Parts:
- added LOGO1: CC-BY-SA_0.33in, Symbol_CreativeCommons:CC-BY-SA_SilkScreenTop_Small, B.Cu at (115.0, 125.0)
