File: banana2header.kicad_pcb (KiCad board)
At the start: 2 copper layers, 35 x 50 mm, 7 parts, among them J1 Conn_01x01_Female, J2 Conn_01x01_Female, J3 Conn_01x01_Female, J4 Molex_SL_01x03_Male, J5 Conn_01x02_Male, J6 Conn_01x02_Male

Commit message: add jlc order number string
Other:
- board text added: "JLCJLCJLCJLC"
Changed lines of the file:
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@@
     (effects (font (size 1.5 1.5) (thickness 0.3)) (justify left mirror))
+  )
+  (gr_text "JLCJLCJLCJLC" (at 97 95 -90) (layer "F.SilkS")
+    (effects (font (size 1 1) (thickness 0.15)))
   )
   (gr_text "BANANA TO PINHEADER" (at 112.5 87) (layer "F.SilkS")
